File: Minibar/PCB/KiCad/Minibar_Strum_Board/Minibar_Strum_Board.kicad_sch (KiCad schematic)
At the start: 23 parts, among them SW1 MX_SW_solder, SW2 MX_SW_solder, SW3 MX_SW_HS, SW4 MX_SW_HS, U1 ProMicro

Commit message: Updated Minibar strum board
Parts:
- removed SW1, SW2: MX_SW_solder, marbastlib-mx:SW_MX_1u, symbol marbastlib-mx:MX_SW_solder
- removed TP1, TP10, TP11, TP12, TP13, TP14, TP2, TP3, TP4, TP5, TP6, TP7, TP8, TP9: TestPoint, TestPoint:TestPoint_THTPad_D3.0mm_Drill1.5mm, symbol Connector:TestPoint
- removed U1: ProMicro, Keebio-Parts:ArduinoProMicro, symbol keebio:ProMicro
- added J1: Conn_01x09_Pin, Connector_PinHeader_2.54mm:PinHeader_1x09_P2.54mm_Vertical, symbol Connector:Conn_01x09_Pin
- added J2, J4: Conn_01x02_Pin, Connector_PinHeader_2.54mm:PinHeader_1x02_P2.54mm_Vertical, symbol Connector:Conn_01x02_Pin
- added J3: Conn_01x02_Pin, Minibar:Solder_Jumper, symbol Connector:Conn_01x02_Pin
- added SW3, SW4: SW, Button_Switch_SMD:SW_SPST_PTS645, symbol marbastlib-mx:MX_SW_HS
- added U1: KB2040, Minibar:KB2040-SMD, symbol Minibar:KB2040
- added U2: Joystick, Minibar:Joystick, symbol Minibar:Joystick
- SW1: renamed from SW3; footprint marbastlib-mx:SW_MX_HS_1u -> Minibar:Kailh_Hotswap_MX
- SW2: renamed from SW4; footprint marbastlib-mx:SW_MX_HS_1u -> Minibar:Kailh_Hotswap_MX
- renumbered D2 to D1, D1 to D2
Connections:
- net Blue: now also J1.4 (Pin_4), U1.14 (16/PB2)
- net Down: now also SW1.1, U1.12 (9/PB5); no longer SW1.2
- net GND: now also D3.3 (GND), D4.3 (GND), SW1.2, SW2.2, J1.6 (Pin_6), J4.2 (Pin_2), SW3.2, SW4.2, U1.23 (GND), U1.3 (GND), U1.4 (GND), U2.B2, U2.VR11, U2.VR21; no longer SW1.1, SW2.1
- net Green: now also J1.1 (Pin_1), U1.17 (A0/PF7)
- net Orange: now also J1.5 (Pin_5), U1.13 (10/PB6)
- net Red: now also J1.2 (Pin_2), U1.16 (15/PB1)
- net SW: now also U1.5 (2/PD1), U2.B1
- net Select: now also SW3.1, U1.8 (5/PC6)
- net Start: now also SW4.1, U1.7 (4/PD4)
- net Up: now also SW2.1, U1.11 (8/PB4); no longer SW2.2
- net VCC: now also J1.7 (Pin_7), U1.21 (VCC), U2.VR13, U2.VR23
- net VRX: now also U1.19 (A2/PF5), U2.VR12
- net VRY: now also U1.18 (A1/PF6), U2.VR22
- net Yellow: now also J1.3 (Pin_3), U1.15 (14/PB3)
- net fret_mosi: now also D1.6 (DO), J1.9 (Pin_9); no longer D4.6 (DO)
- net fret_sck: now also D1.5 (CO), J1.8 (Pin_8); no longer D4.5 (CO)
- net led_mosi: now also D4.1 (DI), U1.6 (3/PD0); no longer D1.1 (DI)
- net led_sck: now also D4.2 (CI), U1.9 (6/PD7); no longer D1.2 (CI)
- net at D3.6 (DO): now also D2.1 (DI); no longer D4.1 (DI)
- net at D3.5 (CO): now also D2.2 (CI); no longer D4.2 (CI)
- net at D3.1 (DI): now also D4.6 (DO); no longer D2.6 (DO)
- net at D3.2 (CI): now also D4.5 (CO); no longer D2.5 (CO)
- new net: D1.2 (CI), D2.5 (CO)
- new net: D1.1 (DI), D2.6 (DO)
- new net Tilt: J2.1 (Pin_1), J3.1 (Pin_1), U1.10 (7/PE6)
- new net Tilt 2: J2.2 (Pin_2), J3.2 (Pin_2), J4.1 (Pin_1)
Other:
- moved on the sheet: D1, SW1, SW2
